Commit message: force based controller

File: src/robbie/urdf/robbie.xacro (robot description, xacro)
@@ -13,5 +13,5 @@
   <xacro:property name="chassis_length" value="0.2"/>
   <xacro:property name="chassis_height" value="0.05"/>
-  <xacro:property name="chassis_mass" value="0.5"/>
+  <xacro:property name="chassis_mass" value="1000000"/>
   <xacro:property name="wheel_radius" value="0.04"/>
   <xacro:property name="wheel_width" value="0.03"/>
@@ -193,7 +193,4 @@
     </plugin>
   </gazebo> -->
-  <gazebo reference="chassis">
-    <gravity>0</gravity>
-  </gazebo>
   <gazebo reference="camera_link">
     <sensor type="camera" name="camera1">

Commit message: added PID controller to twistflyplugin

File: src/robbie/urdf/robbie.xacro (robot description, xacro)
@@ -13,5 +13,5 @@
   <xacro:property name="chassis_length" value="0.2"/>
   <xacro:property name="chassis_height" value="0.05"/>
-  <xacro:property name="chassis_mass" value="1000000"/>
+  <xacro:property name="chassis_mass" value="19.5"/>
   <xacro:property name="wheel_radius" value="0.04"/>
   <xacro:property name="wheel_width" value="0.03"/>

Commit message: Added height sensors, experiment with parallax correction, and fixed clueboard detection

File: src/robbie/urdf/robbie.xacro (robot description, xacro)
@@ -36,62 +36,12 @@
     </visual>
   </link>
-  <link name='wheel_FR'>
-    <xacro:cylinder_inertial name="wheel_FR" m="${wheel_mass}" r="${wheel_radius}" h="${wheel_width}"/>
-    <collision name='wheel_FR_collision'>
-      <origin xyz="0 0 0" rpy="1.5708 0 0"/>
+  <!-- Lidar Link -->
+  <link name="lidar_link">
+    <visual>
+      <origin xyz="0 0 0" rpy="0 0 0"/>
       <geometry>
-        <cylinder radius="${wheel_radius}" length="${wheel_width}"/>
+        <box size="0.02 0.02 0.02"/>
       </geometry>
-    </collision>
-    <visual name='wheel_FR_visual'>
-      <origin xyz="0 0 0" rpy="1.5708 0 0"/>
-      <geometry>
-        <cylinder radius="${wheel_radius}" length="${wheel_width}"/>
-      </geometry>
-    </visual>
-  </link>
-  <link name='wheel_FL'>
-    <xacro:cylinder_inertial name="wheel_FL" m="${wheel_mass}" r="${wheel_radius}" h="${wheel_width}"/>
-    <collision name='wheel_FL_collision'>
-      <origin xyz="0 0 0" rpy="1.5708 0 0"/>
-      <geometry>
-        <cylinder radius="${wheel_radius}" length="${wheel_width}"/>
-      </geometry>
-    </collision>
-    <visual name='wheel_FL_visual'>
-      <origin xyz="0 0 0" rpy="1.5708 0 0"/>
-      <geometry>
-        <cylinder radius="${wheel_radius}" length="${wheel_width}"/>
-      </geometry>
-    </visual>
-  </link>
-  <link name='wheel_RR'>
-    <xacro:cylinder_inertial name="wheel_RR" m="${wheel_mass}" r="${wheel_radius}" h="${wheel_width}"/>
-    <collision name='wheel_RR_collision'>
-      <origin xyz="0 0 0" rpy="1.5708 0 0"/>
-      <geometry>
-        <cylinder radius="${wheel_radius}" length="${wheel_width}"/>
-      </geometry>
-    </collision>
-    <visual name='wheel_RR_visual'>
-      <origin xyz="0 0 0" rpy="1.5708 0 0"/>
-      <geometry>
-        <cylinder radius="${wheel_radius}" length="${wheel_width}"/>
-      </geometry>
-    </visual>
-  </link>
-  <link name='wheel_RL'>
-    <xacro:cylinder_inertial name="wheel_RL" m="${wheel_mass}" r="${wheel_radius}" h="${wheel_width}"/>
-    <collision name='wheel_RL_collision'>
-      <origin xyz="0 0 0" rpy="1.5708 0 0"/>
-      <geometry>
-        <cylinder radius="${wheel_radius}" length="${wheel_width}"/>
-      </geometry>
-    </collision>
-    <visual name='wheel_RL_visual'>
-      <origin xyz="0 0 0" rpy="1.5708 0 0"/>
-      <geometry>
-        <cylinder radius="${wheel_radius}" length="${wheel_width}"/>
-      </geometry>
+      <material name="yellow"/>
     </visual>
   </link>
@@ -116,5 +66,5 @@
         <cylinder radius="0.05" length="0.01"/>
       </geometry>
-      <material name="yellow"/>
+      <material name="black"/>
     </visual>
   </link>
@@ -124,36 +74,13 @@
     <origin xyz="${chassis_length} 0 ${chassis_height/2}" rpy="0 0 0"/>
   </joint>
-  <joint name="wheel_FR_joint" type="continuous">
-    <parent link="chassis"/>
-    <child link="wheel_FR"/>
-    <origin xyz="${chassis_length/2-wheel_radius} -${chassis_width/2+wheel_width/2} 0"
-            rpy="0 0 0"/>
-    <axis xyz="0 1 0"/>
-  </joint>
-  <joint name="wheel_FL_joint" type="continuous">
-    <parent link="chassis"/>
-    <child link="wheel_FL"/>
-    <origin xyz="${chassis_length/2-wheel_radius} ${chassis_width/2+wheel_width/2} 0"
-            rpy="0 0 0"/>
-    <axis xyz="0 1 0"/>
-  </joint>
-  <joint name="wheel_RR_joint" type="continuous">
-    <parent link="chassis"/>
-    <child link="wheel_RR"/>
-    <origin xyz="-${chassis_length/2-wheel_radius} -${chassis_width/2+wheel_width/2} 0"
-            rpy="0 0 0"/>
-    <axis xyz="0 1 0"/>
-  </joint>
-  <joint name="wheel_RL_joint" type="continuous">
-    <parent link="chassis"/>
-    <child link="wheel_RL"/>
-    <origin xyz="-${chassis_length/2-wheel_radius} ${chassis_width/2+wheel_width/2} 0"
-            rpy="0 0 0"/>
-    <axis xyz="0 1 0"/>
-  </joint>
   <joint name="camera_joint" type="fixed">
     <parent link="chassis"/>
     <child link="camera_link"/>
     <origin xyz="0 0 -${chassis_height/2 + camera_height/2}" rpy="0 1.5708 0"/>
+  </joint>
+  <joint name="lidar_joint" type="fixed">
+    <parent link="chassis"/>
+    <child link="lidar_link"/>
+    <origin xyz="0 0.02 -${chassis_height/3+0.01}" rpy="0 1.5708 0"/>
   </joint>
   <gazebo reference="chassis">
@@ -163,18 +90,9 @@
     <material>Gazebo/Blue</material>
   </gazebo>
-  <gazebo reference="wheel_FL">
-    <material>Gazebo/Blue</material>
-  </gazebo>
-  <gazebo reference="wheel_FR">
-    <material>Gazebo/Blue</material>
-  </gazebo>
-  <gazebo reference="wheel_RL">
-    <material>Gazebo/Blue</material>
-  </gazebo>
-  <gazebo reference="wheel_RR">
-    <material>Gazebo/Blue</material>
-  </gazebo>
   <gazebo reference="circle_link">
     <material>Gazebo/Yellow</material>
+  </gazebo>
+  <gazebo reference="lidar_link">
+    <material>Gazebo/Black</material>
   </gazebo>
   <!-- <gazebo>
@@ -195,5 +113,5 @@
   <gazebo reference="camera_link">
     <sensor type="camera" name="camera1">
-      <update_rate>30.0</update_rate>
+      <update_rate>40.0</update_rate>
       <camera name="head">
         <horizontal_fov>1.5</horizontal_fov>
@@ -232,4 +150,44 @@
     </sensor>
   </gazebo>
+  <!-- Lidar -->
+  <gazebo reference="lidar_link">
+    <sensor type="ray" name="height_sensor">
+      <pose>0 0 0 0 0 0</pose>
+      <visualize>true</visualize>
+      <update_rate>30.0</update_rate>
+      <ray>
+        <scan>
+          <horizontal>
+            <samples>50</samples>
+            <resolution>1</resolution>
+            <min_angle>-0.1</min_angle>
+            <max_angle>0.1</max_angle>
+          </horizontal>
+          <vertical>
+            <samples>50</samples>
+            <resolution>1</resolution>
+            <min_angle>-0.1</min_angle>
+            <max_angle>0.1</max_angle>
+          </vertical>
+        </scan>
+        <range>
+          <min>0.05</min>
+          <max>50.0</max>
+          <resolution>0.01</resolution>
+        </range>
+        <noise>
+          <type>gaussian</type>
+          <mean>0.0</mean>
+          <stddev>0.01</stddev>
+        </noise>
+      </ray>
+      <plugin name="ros_ray_sensor_controller" filename="libgazebo_ros_laser.so">
+        <alwaysOn>true</alwaysOn>
+        <updateRate>0.0</updateRate>
+        <topicName>rrbot/height</topicName>
+        <frameName>lidar_link</frameName>
+      </plugin>
+    </sensor>
+  </gazebo>
   <gazebo>
       <plugin name="twistflyplugin" filename="libtwistflyplugin.so">

Commit message: Sign to sign

File: src/robbie/urdf/robbie.xacro (robot description, xacro)
@@ -77,5 +77,5 @@
     <parent link="chassis"/>
     <child link="camera_link"/>
-    <origin xyz="0 0 -${chassis_height/2 + camera_height/2}" rpy="0 1.5708 0"/>
+    <origin xyz="0 0 -${chassis_height/2 + camera_height/2}" rpy="${camera_orientation}"/>
   </joint>
   <joint name="lidar_joint" type="fixed">

Commit message: Specify lidar samples and angles from launch file

File: src/robbie/urdf/robbie.xacro (robot description, xacro)
@@ -5,4 +5,6 @@
   <xacro:property name="robot_name" value="$(arg robot_name)"/>
   <xacro:property name="camera_orientation" value="$(arg camera_orientation)"/>
+  <xacro:property name="lidar_samples" value="$(arg lidar_samples)"/>
+  <xacro:property name="lidar_angle" value="$(arg lidar_angle)"/>
   <!-- <xacro:property name="chassis_colour" value="$(arg chassis_colour)"/> -->
   <xacro:property name="camera_width" value="0.02"/>
@@ -159,14 +161,14 @@
         <scan>
           <horizontal>
-            <samples>50</samples>
+            <samples>${lidar_samples}</samples>
             <resolution>1</resolution>
-            <min_angle>-0.1</min_angle>
-            <max_angle>0.1</max_angle>
+            <min_angle>${-lidar_angle}</min_angle>
+            <max_angle>${lidar_angle}</max_angle>
           </horizontal>
           <vertical>
-            <samples>50</samples>
+            <samples>${lidar_samples}</samples>
             <resolution>1</resolution>
-            <min_angle>-0.1</min_angle>
-            <max_angle>0.1</max_angle>
+            <min_angle>${-lidar_angle}</min_angle>
+            <max_angle>${lidar_angle}</max_angle>
           </vertical>
         </scan>

Commit message: Got clueboard reading working, and delete second target if first one yeilds a clue, finally moved lidar out of camera view

File: src/robbie/urdf/robbie.xacro (robot description, xacro)
@@ -84,5 +84,5 @@
     <parent link="chassis"/>
     <child link="lidar_link"/>
-    <origin xyz="0 0.02 -${chassis_height/3+0.01}" rpy="0 1.5708 0"/>
+    <origin xyz="0 0.02 -${chassis_height/4+0.01}" rpy="0 1.5708 0"/>
   </joint>
   <gazebo reference="chassis">

Commit message: parallel axis correction

File: src/robbie/urdf/robbie.xacro (robot description, xacro)
@@ -48,4 +48,14 @@
     </visual>
   </link>
+    <!-- IMU link -->
+  <link name="imu_link">
+    <visual>
+      <origin xyz="0 0 0" rpy="0 0 0"/>
+      <geometry>
+        <box size="0.02 0.02 0.02"/>
+      </geometry>
+      <material name="yellow"/>
+    </visual>
+  </link>
   <link name='camera_link'>
     <xacro:box_inertial name="camera_link" m="${camera_mass}" x="${camera_width}" y="${camera_length}" z="${camera_height}"/>
@@ -86,4 +96,9 @@
     <origin xyz="0 0.02 -${chassis_height/3+0.01}" rpy="0 1.5708 0"/>
   </joint>
+  <joint name="imu_joint" type="fixed">
+    <parent link="chassis"/>
+    <child link="imu_link"/>
+    <origin xyz="0 0.02 -${chassis_height/3}" rpy="0 0 0"/>
+  </joint>
   <gazebo reference="chassis">
     <material>Gazebo/Orange</material>
@@ -96,4 +111,7 @@
   </gazebo>
   <gazebo reference="lidar_link">
+    <material>Gazebo/Black</material>
+  </gazebo>
+  <gazebo reference="imu_link">
     <material>Gazebo/Black</material>
   </gazebo>
@@ -195,4 +213,24 @@
     </sensor>
   </gazebo>
+  <gazebo reference="imu_link">
+    <gravity>true</gravity>
+    <sensor name="imu_sensor" type="imu">
+      <always_on>true</always_on>
+      <update_rate>100</update_rate>
+      <visualize>true</visualize>
+      <topic>rrbot/imu</topic>
+      <plugin filename="libgazebo_ros_imu_sensor.so" name="imu_plugin">
+        <topicName>imu</topicName>
+        <bodyName>imu_link</bodyName>
+        <updateRateHZ>10.0</updateRateHZ>
+        <gaussianNoise>0.0</gaussianNoise>
+        <xyzOffset>0 0 0</xyzOffset>
+        <rpyOffset>0 0 0</rpyOffset>
+        <frameName>imu_link</frameName>
+        <initialOrientationAsReference>true</initialOrientationAsReference>
+      </plugin>
+      <pose>0 0 0 0 0 0</pose>
+    </sensor>
+  </gazebo>
   <gazebo>
       <plugin name="twistflyplugin" filename="libtwistflyplugin.so">

Commit message: working commit

File: src/robbie/urdf/robbie.xacro (robot description, xacro)
@@ -94,5 +94,5 @@
     <parent link="chassis"/>
     <child link="lidar_link"/>
-    <origin xyz="0 0.02 -${chassis_height/4+0.01}" rpy="0 1.5708 0"/>
+    <origin xyz="${chassis_length/2} 0.02 -${chassis_height/4}" rpy="0 1.5708 0"/>
   </joint>
   <joint name="imu_joint" type="fixed">
